File: Power distribution board.kicad_pcb (KiCad board)
At the start: 2 copper layers, 29.2 x 94 mm, 20 parts, among them P1 CONN_1, P10 CONN_1, P2 CONN_1, P3 CONN_1, P4 CONN_1, P5 CONN_1, P6 CONN_1, P7 CONN_1, P8 CONN_1, P9 CONN_1

Commit message: Fixed silkscreen
Parts:
- moved N2 165.3 mm to (28.4, 98.9)
- moved N3 165.3 mm to (36.0, 98.9)
- moved N1 165.3 mm to (28.4, 107.8)
- moved N10 165.3 mm to (28.4, 27.8)
- moved N4 165.3 mm to (28.4, 81.1)
- moved N5 165.3 mm to (36.0, 81.1)
- moved N6 165.3 mm to (28.4, 63.4)
- moved N7 165.3 mm to (36.0, 63.4)
- moved N8 165.3 mm to (28.4, 45.6)
- moved N9 165.3 mm to (36.0, 45.6)
- moved P1 165.3 mm to (36.0, 107.8)
- moved P10 165.3 mm to (36.0, 27.8)
- moved P2 165.3 mm to (28.4, 90.0)
- moved P3 165.3 mm to (36.0, 90.0)
- moved P4 165.3 mm to (28.4, 72.2)
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
Commit message: Removed battery label for more universal outlook
Other:
- board text removed: "Battery"
Changed lines of the file:
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@@
     (links 18)
     (no_connects 0)
-    (area 16.434999 182.075001 58.982143 280.745001)
+    (area 19.434999 16.825001 61.982143 115.495001)
     (thickness 1.6)
-    (drawings 54)
+    (drawings 50)
     (tracks 28)
     (zones 0)
@@
   )
   (gr_line (start 20.8026 21.4376) (end 22.0472 21.4376) (angle 90) (layer Edge.Cuts) (width 0.15))
-  (gr_text Battery (at 32.25 112.25) (layer F.SilkS)
-    (effects (font (size 1 0.5) (thickness 0.1)))
-  )
   (gr_circle (center 40.86 98.75) (end 42.01 98.16) (layer F.SilkS) (width 0.2))
   (gr_text - (at 40.86 98.7) (layer F.SilkS)
@@
   )
   (gr_circle (center 40.86 90) (end 42.01 89.41) (layer F.SilkS) (width 0.2))
-  (gr_circle (center 36 112.3) (end 37.15 111.71) (layer F.SilkS) (width 0.2))
-  (gr_circle (center 28.39 112.3) (end 29.55 111.75) (layer F.SilkS) (width 0.2))
-  (gr_text - (at 28.4 112.25) (layer F.SilkS)
-    (effects (font (size 2 2) (thickness 0.3)))
-  )
-  (gr_text + (at 36 112.25) (layer F.SilkS)
-    (effects (font (size 2 2) (thickness 0.3)))
-  )
-  (dimension 4 (width 0.25) (layer Dwgs.User)
-    (gr_text "4,000 mm" (at 57.999999 107.750001 270) (layer Dwgs.User)
-      (effects (font (size 1 1) (thickness 0.25)))
-    )
-    (feature1 (pts (xy 38 109.75) (xy 58.999999 109.750001)))
-    (feature2 (pts (xy 38 105.75) (xy 58.999999 105.750001)))
-    (crossbar (pts (xy 56.999999 105.750001) (xy 56.999999 109.750001)))
-    (arrow1a (pts (xy 56.999999 109.750001) (xy 56.413579 108.623498)))
-    (arrow1b (pts (xy 56.999999 109.750001) (xy 57.586419 108.623498)))
-    (arrow2a (pts (xy 56.999999 105.750001) (xy 56.413579 106.876504)))
-    (arrow2b (pts (xy 56.999999 105.750001) (xy 57.586419 106.876504)))
-  )
-  (dimension 93.98 (width 0.25) (layer Dwgs.User)
-    (gr_text "93,980 mm" (at 52.259994 68.43 270) (layer Dwgs.User)
-      (effects (font (size 1 1) (thickness 0.25)))
-    )
-    (feature1 (pts (xy 48.72 115.42) (xy 53.259994 115.42)))
-    (feature2 (pts (xy 48.72 21.44) (xy 53.259994 21.44)))
-    (crossbar (pts (xy 51.259994 21.44) (xy 51.259994 115.42)))
-    (arrow1a (pts (xy 51.259994 115.42) (xy 50.673574 114.293497)))
-    (arrow1b (pts (xy 51.259994 115.42) (xy 51.846414 114.293497)))
-    (arrow2a (pts (xy 51.259994 21.44) (xy 50.673574 22.566503)))
-    (arrow2b (pts (xy 51.259994 21.44) (xy 51.846414 22.566503)))
-  )
-  (dimension 29.21 (width 0.25) (layer Dwgs.User)
-    (gr_text "29,210 mm" (at 34.115 17.900001) (layer Dwgs.User)
-      (effects (font (size 1 1) (thickness 0.25)))
-    )
-    (feature1 (pts (xy 19.51 22.71) (xy 19.51 16.900001)))
-    (feature2 (pts (xy 48.72 22.71) (xy 48.72 16.900001)))
-    (crossbar (pts (xy 48.72 18.900001) (xy 19.51 18.900001)))
-    (arrow1a (pts (xy 19.51 18.900001) (xy 20.636503 18.313581)))
-    (arrow1b (pts (xy 19.51 18.900001) (xy 20.636503 19.486421)))
-    (arrow2a (pts (xy 48.72 18.900001) (xy 47.593497 18.313581)))
-    (arrow2b (pts (xy 48.72 18.900001) (xy 47.593497 19.486421)))
+  (gr_circle (center 40.9 107.806) (end 42.05 107.216) (layer F.SilkS) (width 0.2))
+  (gr_circle (center 23.44 107.725) (end 24.6 107.175) (layer F.SilkS) (width 0.2))
+  (gr_text - (at 23.45 107.675) (layer F.SilkS)
+    (effects (font (size 2 2) (thickness 0.3)))
+  )
+  (gr_text + (at 40.9 107.756) (layer F.SilkS)
+    (effects (font (size 2 2) (thickness 0.3)))
   )
   (gr_line (start 22.05 21.44) (end 47.45 21.44) (angle 90) (layer Edge.Cuts) (width 0.15))
